Commit message: Add base footprint and mock odom TF

File: ros2_ws/src/amr_description/urdf/amr.urdf (robot description, URDF)
Before this commit: robot amr, 5 links, 4 joints
Links:
- added link base_footprint
Joints:
- added joint base_footprint_joint: type fixed, parent base_footprint, child base_link, origin xyz=0 0 0.05 rpy=0 0 0
